File: hardware/nRF54L_ePaper.kicad_pcb (KiCad board)
At the start: 4 copper layers, 58 x 35 mm, 41 parts, among them J1 Conn_01x04, J2 Conn_01x24_MountingPin, J4 Conn_ARM_SWD_TagConnect_TC203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, Q1 Q_NMOS_GSD, Q2 Q_NMOS_GSD, SW1 SW_Push, SW2 SW_Push, SW3 SW_Push, SW4 SW_Push, SW5 SW_SPDT, U1 BM15x, U2 SHT4x, Y2 32.768KHz

Commit message: Updated Dec23/24
Routing:
- net GND: vias 30 -> 33

Commit message: Added button 3D model
Parts:
- SW1, SW2, SW3, SW4: footprint Button_Switch_SMD:SW_Push_1P1T_NO_Vertical_Wuerth_434133025816 -> ePaper54L-Button_Switch_SMD:SW_Push_1P1T_NO_Vertical_Wuerth_434133025816
